Commit message: sample moveit description file 생성 완료

File: robot/strawberry_description/urdf/berry_good_bot_sampleURDF.xacro (robot description, xacro)
@@ -36,5 +36,5 @@
     <origin xyz="0 0 0" rpy="0 0 0"/>
     <axis xyz="0 0 1"/>
-    <limit lower="0.0" upper="1.0" velocity="0.3" effort="100"/>
+    <limit lower="0.0" upper="1.0" velocity="0.3" effort="100.0"/>
   </joint>
   <!-- 3-DOF 팔 -->
@@ -45,5 +45,5 @@
     <origin xyz="0 0 0" rpy="0 0 0"/>
     <axis  xyz="0 0 1"/>
-    <limit lower="-${pi}" upper="${pi}" velocity="1.5" effort="50"/>
+    <limit lower="-${pi}" upper="${pi}" velocity="1.5" effort="50.0"/>
   </joint>
   <xacro:cyl_link name="link2" length="${L2}" radius="${link_radius}"/>
@@ -53,5 +53,5 @@
     <origin xyz="${L1} 0 0" rpy="0 0 0"/>
     <axis  xyz="0 0 1"/>
-    <limit lower="-${pi}" upper="${pi}" velocity="1.5" effort="40"/>
+    <limit lower="-${pi}" upper="${pi}" velocity="1.5" effort="40.0"/>
   </joint>
   <xacro:cyl_link name="link3" length="${L3}" radius="${link_radius}"/>
@@ -61,5 +61,5 @@
     <origin xyz="${L2} 0 0" rpy="0 0 0"/>
     <axis  xyz="0 0 1"/>
-    <limit lower="-${pi}" upper="${pi}" velocity="2.0" effort="30"/>
+    <limit lower="-${pi}" upper="${pi}" velocity="2.0" effort="30.0"/>
   </joint>
   <!-- EEF 축 회전 -->
@@ -70,5 +70,5 @@
     <origin xyz="${L3} 0 0" rpy="0 0 0"/>
     <axis  xyz="1 0 0"/>
-    <limit effort="10" velocity="2.5"/>
+    <limit effort="10.0" velocity="2.5"/>
   </joint>
   <!-- 그리퍼 -->
@@ -79,5 +79,5 @@
     <origin xyz="0 0 0" rpy="0 0 0"/>
     <axis  xyz="0 1 0"/>
-    <limit lower="0.0" upper="0.04" velocity="0.02" effort="20"/>
+    <limit lower="0.0" upper="0.04" velocity="0.02" effort="20.0"/>
   </joint>
   <!-- 작업 좌표계 -->

Commit message: berry_kinematics control 개발중

File: robot/strawberry_description/urdf/berry_good_bot_sampleURDF.xacro (robot description, xacro)
@@ -65,10 +65,13 @@
   <!-- EEF 축 회전 -->
   <link  name="wrist_link"/>
-  <joint name="wrist_roll_joint" type="continuous">
+  <joint name="wrist_roll_joint" type="revolute">
     <parent link="link3"/>
     <child  link="wrist_link"/>
     <origin xyz="${L3} 0 0" rpy="0 0 0"/>
     <axis  xyz="1 0 0"/>
-    <limit effort="10.0" velocity="2.5"/>
+    <limit lower="-3.141592653589793"
+           upper="3.141592653589793"
+           effort="10.0"
+           velocity="2.5"/>
   </joint>
   <!-- 그리퍼 -->
